File: hardware/kicad/Keyboard_LED_button.kicad_sch (KiCad schematic)
At the start: 24 parts, among them J1 JST 4 Pin Qwiic I2C Connector, J2 JST 4 Pin Qwiic I2C Connector, J3 noknok_FlashPads_I2C-module, SW1 SW_Push, U1 CH32V003F4U6, U2 MT3540‑F23

Commit message: hardware: update KiCad layout and schematic, consolidate schematic PDF and fix readme link
Other:
- note removed: "Specs: - I2C powered at 3.3V"
